File: kicad/hp-ref.kicad_pcb (KiCad board)
At the start: 2 copper layers, 49.5 x 42.5 mm, 46 parts, among them J400 CONN_5X1, J401 CONN_5X1, Q401 MJE182, U401 LTZ1000A, U402 LT1013, X411 15k, X411412 15k / 1k, X412 1k, X414 111R

Commit message: fixing test point solder masks
Parts:
- TEST_SMD_05 (x7): moved to F.Cu
Changed lines of the file:
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@@
     (links 75)
     (no_connects 0)
-    (area 183.464999 118.694999 233.095001 161.975001)
+    (area 182.498999 118.618 245.93006 161.340001)
     (thickness 1.6)
     (drawings 16)
@@
     )
   )
-  (module TEST_SMD_02 (layer B.Cu)
+  (module TEST_SMD_02 (layer F.Cu)
     (at 231.14 122.555)
     (descr "Test point, SMD, 0.05\"")
-    (fp_text reference TEST_SMD_05 (at 0 -1.905) (layer B.SilkS) hide
-      (effects (font (size 0.762 0.762) (thickness 0.1524)) (justify mirror))
-    )
-    (fp_text value VAL** (at 0 1.905) (layer B.SilkS) hide
-      (effects (font (size 1 1) (thickness 0.15)) (justify mirror))
+    (fp_text reference TEST_SMD_05 (at 0 1.905) (layer F.SilkS) hide
+      (effects (font (size 0.762 0.762) (thickness 0.1524)))
+    )
+    (fp_text value VAL** (at 0 -1.905) (layer F.SilkS) hide
+      (effects (font (size 1 1) (thickness 0.15)))
     )
     (pad 1 smd circle (at 0 0) (size 1.27 1.27)
@@
     )
   )
-  (module TEST_SMD_02 (layer B.Cu)
+  (module TEST_SMD_02 (layer F.Cu)
     (at 231.14 125.095)
     (descr "Test point, SMD, 0.05\"")
-    (fp_text reference TEST_SMD_05 (at 0 -1.905) (layer B.SilkS) hide
-      (effects (font (size 0.762 0.762) (thickness 0.1524)) (justify mirror))
-    )
-    (fp_text value VAL** (at 0 1.905) (layer B.SilkS) hide
-      (effects (font (size 1 1) (thickness 0.15)) (justify mirror))
+    (fp_text reference TEST_SMD_05 (at 0 1.905) (layer F.SilkS) hide
+      (effects (font (size 0.762 0.762) (thickness 0.1524)))
+    )
+    (fp_text value VAL** (at 0 -1.905) (layer F.SilkS) hide
+      (effects (font (size 1 1) (thickness 0.15)))
     )
     (pad 1 smd circle (at 0 0) (size 1.27 1.27)
@@
     )
   )
-  (module TEST_SMD_02 (layer B.Cu)
+  (module TEST_SMD_02 (layer F.Cu)
     (at 215.9 125.095)
     (descr "Test point, SMD, 0.05\"")
-    (fp_text reference TEST_SMD_05 (at 0 -1.905) (layer B.SilkS) hide
-      (effects (font (size 0.762 0.762) (thickness 0.1524)) (justify mirror))
-    )
-    (fp_text value VAL** (at 0 1.905) (layer B.SilkS) hide
-      (effects (font (size 1 1) (thickness 0.15)) (justify mirror))
+    (fp_text reference TEST_SMD_05 (at 0 1.905) (layer F.SilkS) hide
+      (effects (font (size 0.762 0.762) (thickness 0.1524)))
+    )
+    (fp_text value VAL** (at 0 -1.905) (layer F.SilkS) hide
+      (effects (font (size 1 1) (thickness 0.15)))
     )
     (pad 1 smd circle (at 0 0) (size 1.27 1.27)
@@
     )
   )
-  (module TEST_SMD_02 (layer B.Cu)
+  (module TEST_SMD_02 (layer F.Cu)
     (at 213.36 122.555)
     (descr "Test point, SMD, 0.05\"")
-    (fp_text reference TEST_SMD_05 (at 0 -1.905) (layer B.SilkS) hide
-      (effects (font (size 0.762 0.762) (thickness 0.1524)) (justify mirror))
-    )
-    (fp_text value VAL** (at 0 1.905) (layer B.SilkS) hide
-      (effects (font (size 1 1) (thickness 0.15)) (justify mirror))
+    (fp_text reference TEST_SMD_05 (at 0 1.905) (layer F.SilkS) hide
+      (effects (font (size 0.762 0.762) (thickness 0.1524)))
+    )
+    (fp_text value VAL** (at 0 -1.905) (layer F.SilkS) hide
+      (effects (font (size 1 1) (thickness 0.15)))
     )
     (pad 1 smd circle (at 0 0) (size 1.27 1.27)
@@
     )
     (pad 1 smd circle (at 0 0) (size 1.27 1.27)
-      (layers B.Cu F.Paste F.Mask)
+      (layers B.Cu B.Paste B.Mask)
       (net 2 +18H)
     )
@@
     )
     (pad 1 smd circle (at 0 0) (size 1.27 1.27)
-      (layers B.Cu F.Paste F.Mask)
+      (layers B.Cu B.Paste B.Mask)
       (net 4 -15)
     )
@@
     )
     (pad 1 smd circle (at 0 0) (size 1.27 1.27)
-      (layers B.Cu F.Paste F.Mask)
+      (layers B.Cu B.Paste B.Mask)
       (net 5 "H GND")
     )
@@
     )
     (pad 1 smd circle (at 0 0) (size 1.27 1.27)
-      (layers B.Cu F.Paste F.Mask)
+      (layers B.Cu B.Paste B.Mask)
       (net 1 +18)
     )
@@
     )
     (pad 1 smd circle (at 0 0) (size 1.27 1.27)
-      (layers B.Cu F.Paste F.Mask)
+      (layers B.Cu B.Paste B.Mask)
       (net 8 "J401 (1)")
     )
@@
     )
     (pad 1 smd circle (at 0 0) (size 1.27 1.27)
-      (layers B.Cu F.Paste F.Mask)
+      (layers B.Cu B.Paste B.Mask)
       (net 2 +18H)
     )
   )
-  (module TEST_SMD_02 (layer B.Cu)
+  (module TEST_SMD_02 (layer F.Cu)
     (at 218.44 127.635)
     (descr "Test point, SMD, 0.05\"")
-    (fp_text reference TEST_SMD_05 (at 0 -1.905) (layer B.SilkS) hide
-      (effects (font (size 0.762 0.762) (thickness 0.1524)) (justify mirror))
-    )
-    (fp_text value VAL** (at 0 1.905) (layer B.SilkS) hide
-      (effects (font (size 1 1) (thickness 0.15)) (justify mirror))
+    (fp_text reference TEST_SMD_05 (at 0 1.905) (layer F.SilkS) hide
+      (effects (font (size 0.762 0.762) (thickness 0.1524)))
+    )
+    (fp_text value VAL** (at 0 -1.905) (layer F.SilkS) hide
+      (effects (font (size 1 1) (thickness 0.15)))
     )
     (pad 1 smd circle (at 0 0) (size 1.27 1.27)
@@
     )
     (pad 1 smd circle (at 0 0) (size 1.27 1.27)
-      (layers B.Cu F.Paste F.Mask)
+      (layers B.Cu B.Paste B.Mask)
       (net 6 "J400 (1)")
     )
@@
     )
     (pad 1 smd circle (at 0 0) (size 1.27 1.27)
-      (layers B.Cu F.Paste F.Mask)
+      (layers B.Cu B.Paste B.Mask)
     )
   )
@@
     )
     (pad 1 smd circle (at 0 0) (size 1.27 1.27)
-      (layers B.Cu F.Paste F.Mask)
+      (layers B.Cu B.Paste B.Mask)
       (net 7 "J400 (2)")
     )
@@
     )
     (pad 1 smd circle (at 0 0) (size 1.27 1.27)
-      (layers B.Cu F.Paste F.Mask)
+      (layers B.Cu B.Paste B.Mask)
       (net 3 +7)
     )
@@
     )
     (pad 1 smd circle (at 0 0) (size 1.27 1.27)
-      (layers B.Cu F.Paste F.Mask)
+      (layers B.Cu B.Paste B.Mask)
       (net 9 N-000001)
     )
@@
     )
     (pad 1 smd circle (at 0 0) (size 1.27 1.27)
-      (layers B.Cu F.Paste F.Mask)
+      (layers B.Cu B.Paste B.Mask)
       (net 13 N-000002)
     )
@@
       (xy -1.51384 2.24536)) (layer F.SilkS) (width 0.00254))
   )
-  (module TEST_SMD_02 (layer B.Cu)
+  (module TEST_SMD_02 (layer F.Cu)
     (at 215.9 153.035)
     (descr "Test point, SMD, 0.05\"")
-    (fp_text reference TEST_SMD_05 (at 0 -1.905) (layer B.SilkS) hide
-      (effects (font (size 0.762 0.762) (thickness 0.1524)) (justify mirror))
-    )
-    (fp_text value VAL** (at 0 1.905) (layer B.SilkS) hide
-      (effects (font (size 1 1) (thickness 0.15)) (justify mirror))
+    (fp_text reference TEST_SMD_05 (at 0 1.905) (layer F.SilkS) hide
+      (effects (font (size 0.762 0.762) (thickness 0.1524)))
+    )
+    (fp_text value VAL** (at 0 -1.905) (layer F.SilkS) hide
+      (effects (font (size 1 1) (thickness 0.15)))
     )
     (pad 1 smd circle (at 0 0) (size 1.27 1.27)
@@
     )
   )
-  (module TEST_SMD_02 (layer B.Cu)
+  (module TEST_SMD_02 (layer F.Cu)
     (at 215.9 147.955)
     (descr "Test point, SMD, 0.05\"")
-    (fp_text reference TEST_SMD_05 (at 0 -1.905) (layer B.SilkS) hide
-      (effects (font (size 0.762 0.762) (thickness 0.1524)) (justify mirror))
-    )
-    (fp_text value VAL** (at 0 1.905) (layer B.SilkS) hide
-      (effects (font (size 1 1) (thickness 0.15)) (justify mirror))
+    (fp_text reference TEST_SMD_05 (at 0 1.905) (layer F.SilkS) hide
+      (effects (font (size 0.762 0.762) (thickness 0.1524)))
+    )
+    (fp_text value VAL** (at 0 -1.905) (layer F.SilkS) hide
+      (effects (font (size 1 1) (thickness 0.15)))
     )
     (pad 1 smd circle (at 0 0) (size 1.27 1.27)
@@
   (segment (start 216.535 124.46) (end 213.995 122.555) (width 0.254) (layer F.Cu) (net 5))
   (segment (start 213.995 153.67) (end 201.93 153.67) (width 0.254) (layer B.Cu) (net 6))
-  (segment (start 215.9 153.035) (end 216.535 152.4) (width 0.254) (layer B.Cu) (net 6) (status 400000))
+  (segment (start 215.9 153.035) (end 216.535 152.4) (width 0.254) (layer B.Cu) (net 6))
   (segment (start 221.615 152.4) (end 222.358949 152.291051) (width 0.254) (layer B.Cu) (net 6))
   (segment (start 216.535 152.4) (end 221.615 152.4) (width 0.254) (layer B.Cu) (net 6))

Commit message: fixing molex connector labels
Parts:
- J400, J401: value CONN_5X1 -> 22-17-2052
Changed lines of the file:
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@@
     (18 B.Paste user)
     (19 F.Paste user)
-    (20 B.SilkS user hide)
-    (21 F.SilkS user hide)
+    (20 B.SilkS user)
+    (21 F.SilkS user)
     (22 B.Mask user)
     (23 F.Mask user)
@@
     (pad_to_mask_clearance 0)
     (aux_axis_origin 0 0)
-    (visible_elements FFFFFFAF)
+    (visible_elements FFFFFFBF)
     (pcbplotparams
       (layerselection 284196865)
@@
       (effects (font (size 0.762 0.762) (thickness 0.1524)))
     )
-    (fp_text value CONN_5X1 (at 0 -1.905) (layer F.SilkS)
+    (fp_text value 22-17-2052 (at 0 -1.905) (layer F.SilkS)
       (effects (font (size 0.762 0.762) (thickness 0.1524)))
     )
@@
       (effects (font (size 0.762 0.762) (thickness 0.1524)))
     )
-    (fp_text value CONN_5X1 (at 0 -1.905 180) (layer F.SilkS)
-      (effects (font (size 0.762 0.762) (thickness 0.1524)))
-    )
+    (fp_text value 22-17-2052 (at 0 -1.905 180) (layer F.SilkS)
+      (effects (font (size 0.762 0.762) (thickness 0.1524)))
+    )
